File: hardware/Multi_Board_ASK/Multi_Board_ASK.kicad_pcb (KiCad board)
At the start: 2 copper layers, 76.2 x 53.3 mm, 12 parts, among them J1 Conn_Battery, J2 USB_B_Micro, J3 Conn_Left, J4 Conn_Right, P1 Power, P2 Analog, P3 Digital, P4 Digital

Commit message: Update gitignore
Parts:
- removed REF** (x2): MountingHole_2.5mm_Pad, MountingHole:MountingHole_2.5mm_Pad
- removed REF** (x2): MountingHole_2.2mm_M2, MountingHole:MountingHole_2.2mm_M2
- added J5: Conn_01x02, NANO_FEATHER_R_1:JST-PH_S2B-PH-SM4-TB, F.Cu at (213.2, 113.7)
- added JP1: Jumper_NC_Small, nano_feather_r_1:SolderJumper-2_P1.3mm_Bridged_RoundedPad1.0x1.5mm, B.Cu at (214.5, 83.8)
- added U1: Feather_Cu, NANO_FEATHER_R_1:Feather_CU, F.Cu at (213.9, 70.5)
- added U10: Feather_Silks, NANO_FEATHER_R_1:Moon_The_Shield_SilkS, B.Cu at (213.5, 82.2)
- added U11: KiCadLogo, NANO_FEATHER_R_1:OSHW-Logo2_7.3x6mm_SilkScreen, B.Cu at (213.4, 105.4)
- added U2: Feather_Silks, NANO_FEATHER_R_1:Feather_Silks, F.Cu at (213.1, 90.7)
- added U3: KiCadLogo, NANO_FEATHER_R_1:Ki-2500, F.Cu at (213.3, 86.8)
- added U4: Moon_Firma, NANO_FEATHER_R_1:Moon_Firma_SilkS, F.Cu at (214.1, 96.4)
- added U5: Feather_Silks, NANO_FEATHER_R_1:Moon_The_Shield_SilkS, F.Cu at (213.0, 101.8)
- added U6: KiCadLogo, NANO_FEATHER_R_1:OSHW-Logo2_7.3x6mm_SilkScreen, F.Cu at (212.9, 80.0)
- added U7: Feather_Cu, NANO_FEATHER_R_1:Feather_CU, B.Cu at (213.4, 117.5)
- added U8: KiCadLogo, NANO_FEATHER_R_1:Ki-2500, B.Cu at (213.9, 97.8)
- added U9: Moon_Firma, NANO_FEATHER_R_1:Moon_Firma_SilkS, B.Cu at (214.0, 89.5)
- J1: value Conn_Battery -> feather long; footprint Connector_JST:JST_PH_B2B-PH-SM4-TB_1x02-1MP_P2.00mm_Vertical -> NANO_FEATHER_R_1:PinHeader_1x16_P2.54mm_Vertical; moved to B.Cu
- J2: value USB_B_Micro -> feather short; footprint Connector_USB:USB_Micro-B_Molex-105017-0001 -> NANO_FEATHER_R_1:PinHeader_1x12_P2.54mm_Vertical; moved to B.Cu
- J3: value Conn_Left -> Conn_01x15; footprint Connector_PinSocket_2.54mm:PinSocket_1x16_P2.54mm_Vertical -> NANO_FEATHER_R_1:PinSocket_1x15_P2.54mm_Vertical
- J4: value Conn_Right -> Conn_01x15; footprint Connector_PinSocket_2.54mm:PinSocket_1x12_P2.54mm_Vertical -> NANO_FEATHER_R_1:PinSocket_1x15_P2.54mm_Vertical
- moved J2 88.5 mm to (223.4, 109.9)
- moved J4 80.8 mm to (205.6, 108.6)
- moved J3 75.7 mm to (220.9, 108.6)
- moved J1 74.6 mm to (203.1, 109.9), turned to 0 degrees
Connections:
- net /A5 renamed /D7
- J1 pad 1: GND -> /D2
- J1 pad 2: +BATT -> /TX
- J2 pad 1: VBUS -> /SDA-A4
- J2 pad 2: Net-(J2-Pad2) -> /SCL-A5
- J2 pad 3: Net-(J2-Pad3) -> /D3
- J2 pad 4: Net-(J2-Pad4) -> /D4
- J2 pad 5: GND -> /D5
- J2 pad 6: GND -> /D6
- J3 pad 1: /~RST~ -> /TX
- J3 pad 11: /SCK -> /D8
- J3 pad 12: /MOSI -> /D9
- J3 pad 13: /MISO -> /D10
- J3 pad 14: /RX -> /D11-MOSI
- J3 pad 15: /TX -> /D12-MISO
- J3 pad 2: +3V3 -> /RX
- J3 pad 3: /Aref -> /~RESET
- J3 pad 5: /A0 -> /D2
- J3 pad 6: /A1 -> /D3
- J3 pad 7: /A2 -> /D4
- J3 pad 8: /A3 -> /D5
- J3 pad 9: /A4 -> /D6
- J4 pad 1: +BATT -> /VIN
- J4 pad 10: /GPIO05 -> /A2
- J4 pad 11: /SCL -> /A1
- J4 pad 12: /SDA -> /A0
- J4 pad 2: /EN -> GND
- J4 pad 3: VBUS -> /~RESET
- J4 pad 4: /GPIO13 -> +5V
- J4 pad 5: /GPIO12 -> /A7
- J4 pad 6: /GPIO11 -> /A6
- J4 pad 7: /GPIO10 -> /SCL-A5
- J4 pad 8: /GPIO09 -> /SDA-A4
- J4 pad 9: /GPIO06 -> /A3
Routing:
- net GND: track 0.00 -> 59.0 mm, vias 0 -> 8
- net /~RESET: track 0.00 -> 52.9 mm, vias 0 -> 2
- net /VIN: track 0.00 -> 39.5 mm, vias 0 -> 2
- net /D12-MISO: track 0.00 -> 38.7 mm
- net /D11-MOSI: track 0.00 -> 34.6 mm, vias 0 -> 1
- net /SDA-A4: track 0.00 -> 32.2 mm, vias 0 -> 2
- net /SCK-D13: track 0.00 -> 29.4 mm
- net /SCL-A5: track 0.00 -> 28.4 mm, vias 0 -> 2
- net +5V: track 0.00 -> 26.5 mm, vias 0 -> 3
- net /D2: track 0.00 -> 22.5 mm, vias 0 -> 1
- net /TX: track 0.00 -> 19.1 mm
- net /RX: track 0.00 -> 18.3 mm
- net /D8: track 0.00 -> 16.8 mm, vias 0 -> 2
- net /D9: track 0.00 -> 16.0 mm
- net /D3: track 0.00 -> 12.5 mm
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- added copper zone on B.Cu, net GND
- added copper zone on F.Cu, net GND
Other:
- board size 76.2 x 53.3 mm -> 28.8 x 53.3 mm
- net class Default: clearance 0.2 -> 0.1524; trace_width 0.25 -> 0.1524; via_dia 0.8 -> 0.6; via_drill 0.4 -> 0.3
- net class Power added: clearance 0.1524, trace_width 0.6096, via_dia 0.6858, via_drill 0.3302
- rule pad_to_mask_clearance: 0.051 -> 0.0508
- rule trace_clearance: 0.2 -> 0.1524
- rule trace_min: 0.2 -> 0.1524
- rule via_min_size: 0.4 -> 0.6
- board text added: "+"
- board text added: "-"
- board text added: "VBAT"

Commit message: Add doctos
Parts:
- removed J5: Conn_01x02, NANO_FEATHER_R_1:JST-PH_S2B-PH-SM4-TB
- removed JP1: Jumper_NC_Small, nano_feather_r_1:SolderJumper-2_P1.3mm_Bridged_RoundedPad1.0x1.5mm
- removed U1, U7: Feather_Cu, NANO_FEATHER_R_1:Feather_CU
- removed U10, U5: Feather_Silks, NANO_FEATHER_R_1:Moon_The_Shield_SilkS
- removed U11, U6: KiCadLogo, NANO_FEATHER_R_1:OSHW-Logo2_7.3x6mm_SilkScreen
- removed U2: Feather_Silks, NANO_FEATHER_R_1:Feather_Silks
- removed U3, U8: KiCadLogo, NANO_FEATHER_R_1:Ki-2500
- removed U4, U9: Moon_Firma, NANO_FEATHER_R_1:Moon_Firma_SilkS
- J1: footprint NANO_FEATHER_R_1:PinHeader_1x16_P2.54mm_Vertical -> Multi_Board_ASK:PinHeader_1x16_P2.54mm_Vertical
- J2: footprint NANO_FEATHER_R_1:PinHeader_1x12_P2.54mm_Vertical -> Multi_Board_ASK:PinHeader_1x12_P2.54mm_Vertical
- J3, J4: footprint NANO_FEATHER_R_1:PinSocket_1x15_P2.54mm_Vertical -> Multi_Board_ASK:PinSocket_1x15_P2.54mm_Vertical
- moved J2 91.4 mm to (133.2, 124.5), turned to 270 degrees
- moved J3 87.4 mm to (134.5, 122.0), turned to 90 degrees
- moved J4 71.1 mm to (134.5, 106.8), turned to 90 degrees
- moved J1 70.1 mm to (133.2, 104.2), turned to 270 degrees
- moved P2 56.2 mm to (171.7, 62.9), turned to 90 degrees
- moved P4 53.7 mm to (123.4, 67.9), turned to 90 degrees
- moved P3 36.6 mm to (123.4, 94.9), turned to 90 degrees
- moved P1 34.7 mm to (171.7, 85.7), turned to 90 degrees
Connections:
- net /EN renamed Net-(J2-Pad11)
- net /IOREF renamed Net-(P1-Pad2)
- J1 pad 2: /TX -> /1(Tx)
- J1 pad 3: /RX -> /0(Rx)
- J1 pad 6: /SCK-D13 -> /D13-SCK
- J2 pad 12: Net-(J2-Pad12) -> /VIN
- J2 pad 3: /D3 -> /D3(**)
- J2 pad 5: /D5 -> /D5(**)
- J2 pad 6: /D6 -> /D6(**)
- J2 pad 8: /D9 -> /D9(**)
- J2 pad 9: /D10 -> /D10(**)
- J3 pad 1: /TX -> /1(Tx)
- J3 pad 12: /D9 -> /D9(**)
- J3 pad 13: /D10 -> /D10(**)
- J3 pad 2: /RX -> /0(Rx)
- J3 pad 6: /D3 -> /D3(**)
- J3 pad 8: /D5 -> /D5(**)
- J3 pad 9: /D6 -> /D6(**)
- J4 pad 13: /AREF -> Net-(J4-Pad13)
- J4 pad 15: /SCK-D13 -> /D13-SCK
- P1 pad 3: /Reset -> /~RESET
- P1 pad 8: /Vin -> /VIN
- P2 pad 5: /A4(SDA) -> /SDA-A4
- P2 pad 6: /A5(SCL) -> /SCL-A5
- P3 pad 1: /A5(SCL) -> /SCL-A5
- P3 pad 10: /8 -> /D8
- P3 pad 2: /A4(SDA) -> /SDA-A4
- P3 pad 3: /AREF -> Net-(P3-Pad3)
- P3 pad 5: /13(SCK) -> /D13-SCK
- P3 pad 6: /12(MISO) -> /D12-MISO
- P3 pad 7: /11(**/MOSI) -> /D11-MOSI
- P3 pad 8: /10(**/SS) -> /D10(**)
- P3 pad 9: /9(**) -> /D9(**)
- P4 pad 1: /7 -> /D7
- P4 pad 2: /6(**) -> /D6(**)
- P4 pad 3: /5(**) -> /D5(**)
- P4 pad 4: /4 -> /D4
- P4 pad 5: /3(**) -> /D3(**)
- P4 pad 6: /2 -> /D2
Routing:
- net GND: track 59.0 -> 0.00 mm, vias 8 -> 0
- net /~RESET: track 52.9 -> 0.00 mm, vias 2 -> 0
- net /VIN: track 39.5 -> 0.00 mm, vias 2 -> 0
- net /D12-MISO: track 38.7 -> 0.00 mm
- net /D11-MOSI: track 34.6 -> 0.00 mm, vias 1 -> 0
- net /SDA-A4: track 32.2 -> 0.00 mm, vias 2 -> 0
- net /SCK-D13: track 29.4 -> 0.00 mm
- net /SCL-A5: track 28.4 -> 0.00 mm, vias 2 -> 0
- net +5V: track 26.5 -> 0.00 mm, vias 3 -> 0
- net /D2: track 22.5 -> 0.00 mm, vias 1 -> 0
- net /TX: track 19.1 -> 0.00 mm
- net /RX: track 18.3 -> 0.00 mm
- net /D8: track 16.8 -> 0.00 mm, vias 2 -> 0
- net /D9: track 16.0 -> 0.00 mm
- net /D3: track 12.5 -> 0.00 mm
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Other:
- board size 28.8 x 53.3 mm -> 53.7 x 50.2 mm
- net class Default: clearance 0.1524 -> 0.2; trace_width 0.1524 -> 0.25; via_drill 0.3 -> 0.4
- net class Power removed
- rule pad_to_mask_clearance: 0.0508 -> 0
- rule trace_clearance: 0.1524 -> 0.2
- rule trace_min: 0.1524 -> 0.2
- rule via_min_size: 0.6 -> 0.4
- board text removed: "+"
- board text removed: "-"
- board text removed: "1"
- board text removed: "VBAT"
